Commit message: Trabalho final pt 1

File: urdf/pioneer3dx.xacro (robot description, xacro)
@@ -166,5 +166,5 @@
 	<xacro:p3dx_wheel suffix="right" parent="base_link" reflect="1"/>
 	<!-- front_sonar -->
-	<link name="front_sonar">
+	<!-- <link name="front_sonar">
 		<inertial>
 			<mass value="0.0001" />
@@ -190,7 +190,7 @@
 		<parent link="base_link" />
 		<child link="front_sonar" />
-	</joint>
+	</joint> -->
 	<!-- lms100 laser -->
-	<link name="lms100">
+	<!-- <link name="lms100">
 		<inertial>
 			<mass value="1e-5" />
@@ -216,4 +216,4 @@
 		<parent link="base_link" />
 		<child link="lms100" />
-	</joint>
+	</joint> -->
 </robot>
